File: HW/frontend/RFshield/_saved_Rfshield.sch (KiCad schematic (older format))
At the start: 150 parts, among them P10 TXENABLE, P11 RXENABLE, P12 XTAL2, P13 GCK1, P14 GCK2, P15 SGPIO_CLK, P16 DA0, P17 DA4, P18 DA7, P19 DD0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

Commit message: low budget version of rfshield netlisted
Connections:
- net DD3: no longer PFIO1.14 (P14)
Changed lines of the file:
@@
 Text GLabel 14900 7700 2    40   Input ~ 0
 DD2
-Text GLabel 14900 7600 2    40   Input ~ 0
-DD3
 Text GLabel 14900 7500 2    40   Input ~ 0
 DD4
