File: HW/frontend/RFshield/Rfshield.sch (KiCad schematic (older format))
At the start: 150 parts, among them P10 TXENABLE, P11 RXENABLE, P12 XTAL2, P13 GCK1, P14 GCK2, P15 SGPIO_CLK, P16 DA0, P17 DA4, P18 DA7, P19 DD0, P2 VAA, P20 DD5, P21 DD9, P22 RSSI, P23 GND, P24 GND, P25 GND, P26 GND, P27 GND, P28 GND, P29 GND, P3 SCL, P30 GND, P31 GND, P32 GND, P33 XCVR_CLKOUT, P37 INTR, P38 CLKIN, P39 CLKOUT, P4 SDA, P5 SSP1_SCK, P6 SSP1_MOSI, P7 SSP1_MISO, P8 CS_XCVR, P9 CS_AD, Q1 MOSFET_P, T1 RX_BALUN, T2 TX_BALUN, U1 MAX2837, U2 MAX5864, U3 SI5351C, X1 GSG-XTAL4PIN

Commit message: smd discrete components switched to 0402 package
Parts:
- C19: value 2.2uF -> 100nF
Connections:
- net VAA: now also C11.1, C45.1, C46.1, C57.1, U1.20 (VCCDIG), U2.18 (OVDD); no longer C22.1
- net VCC: now also C22.1; no longer C11.1, C45.1, C46.1, C57.1, U1.20 (VCCDIG), U2.18 (OVDD)

Commit message: ok
Parts:
- added D3, D4, D5: LED, LEDs:LED-3MM, symbol LED
- added R35, R36, R37: 475, hackrf1:GSG-0402, symbol R
Connections:
- net CLK6: now also PFIO2.16 (P16)
- net GCK2: now also PFIO2.22 (P22)
- net GND: now also R35.2, R36.2, R37.2
- net MCU_CLK: now also PFIO2.20 (P20)
- net MIX_CLK: now also PFIO2.18 (P18)
- net RXENABLE: now also D3.2 (A)
- net SGPIO_CLK: now also PFIO2.24 (P24)
- net TXENABLE: now also D4.2 (A)
- net VAA: no longer C57.1
- net VCC: now also C57.1
- net XCVR_EN: now also D5.2 (A)
- net GainCtrl_B1: now reaches U1.12 (B1)
- net GainCtrl_B1: now also PSA1.28 (P28)
- net GainCtrl_B5: now reaches U1.3 (B5)
- net GainCtrl_B5: now also PSA1.20 (P20)
- net GainCtrl_B7: now reaches U1.33 (B7)
- net GainCtrl_B7: now also PSA1.16 (P16)
- net GainCtrl_B6: now reaches U1.34 (B6)
- net GainCtrl_B6: now also PSA1.18 (P18)
- net RXHP: now reaches U1.40 (RXHP)
- net RXHP: now also PSA1.3 (P3)
- net GainCtrl_B4: now reaches U1.6 (B4)
- net GainCtrl_B4: now also PSA1.22 (P22)
- net GainCtrl_B3: now reaches U1.8 (B3)
- net GainCtrl_B3: now also PSA1.24 (P24)
- net GainCtrl_B2: now reaches U1.9 (B2)
- net GainCtrl_B2: now also PSA1.26 (P26)
- new net: D3.1 (K), R35.1
- new net: D5.1 (K), R37.1
- new net: D4.1 (K), R36.1
- no-connect marks 66 -> 45
Other:
- note added: "BYPASS \nBypass with a 1μF \ncapacitor to GND. \nDo not connect other\ncircuitry to this point."
- note added: "VCCRXLNA,\nVCCTXPAD,\nVCCTXMX,\nVCCXTAL,\nVCCDIG\nVCCCP\nBypass with a capacitor \nas close as possible to \nthe pin."
- note removed: "transceiver\n logic pins\n"
- moved on the sheet: C31, C34, C36, C42, L1, L2, L3, L4, PFIO2, T1, T2
