File: HW/frontend/RFshield/Rfshield.sch (KiCad schematic (older format))
At the start: 156 parts, among them P10 TXENABLE, P11 RXENABLE, P12 XTAL2, P13 GCK1, P14 GCK2, P15 SGPIO_CLK, P16 DA0, P17 DA4, P18 DA7, P19 DD0, P2 VAA, P20 DD5, P21 DD9, P22 RSSI, P23 GND, P24 GND, P25 GND, P26 GND, P27 GND, P28 GND, P29 GND, P3 SCL, P30 GND, P31 GND, P32 GND, P33 XCVR_CLKOUT, P37 INTR, P38 CLKIN, P39 CLKOUT, P4 SDA, P5 SSP1_SCK, P6 SSP1_MOSI, P7 SSP1_MISO, P8 CS_XCVR, P9 CS_AD, Q1 MOSFET_P, T1 RX_BALUN, T2 TX_BALUN, U1 MAX2837, U2 MAX5864, U3 SI5351C, X1 GSG-XTAL4PIN

Commit message: all components placed and routed
drc check pending
Parts:
- added C61, C62, C63, C64, C65, C66, C68, C71: 10nF, Capacitors_SMD:C_0402, symbol C
- added C67, C69, C70: 22pF, Capacitors_SMD:C_0402, symbol C
- added P1, P34: CONN_01X01, Connect:GSG-HOLE-06mm1, symbol CONN_01X01
- added R38: 0, Resistors_SMD:R_0402, symbol R
- C11, C8, C9: value 10nF -> 22pF
- C14, C7: value 100nF -> 22pF
- D3, D4, D5: footprint LEDs:LED-3MM -> LEDs:LED-0603
Connections:
- net DD0: now also PFIO1.13 (P13); no longer PFIO1.20 (P20)
- net DD1: now also PFIO1.10 (P10); no longer PFIO1.18 (P18)
- net DD2: now also PFIO1.8 (P8); no longer PFIO1.16 (P16)
- net DD3: now also PFIO1.7 (P7); no longer PFIO1.14 (P14)
- net DD4: now also PFIO1.6 (P6); no longer PFIO1.12 (P12)
- net DD5: now also PFIO1.5 (P5); no longer PFIO1.10 (P10)
- net DD6: now also PFIO1.4 (P4); no longer PFIO1.8 (P8)
- net DD7: now also PFIO1.3 (P3); no longer PFIO1.6 (P6)
- net DD8: now also PFIO1.2 (P2); no longer PFIO1.4 (P4)
- net DD9: now also PFIO1.1 (P1); no longer PFIO1.2 (P2)
- net GND: now also C61.2, C62.2, C63.2, C65.2, C68.2, C69.2, C70.2, C71.2, P1.1 (P1), R38.1; no longer C11.2, C12.2, C13.2, C16.2, C17.2, C18.2, C19.2, C21.2, C22.2, C23.2, C24.2, C28.2, C29.2, C32.2, C44.2, C45.2, C46.2, C47.1, C48.1, C53.2, C54.2, C55.2, C56.2, C57.2, C58.2, C59.2, C60.2, C7.2, D1.1 (A), D2.1 (A), P38.2 (GND), P39.2 (GND), R23.2, U2.0 (EP), U2.12 (GND), U2.17 (OGND), U2.37 (GND), U2.42 (GND), U2.5 (GND), U2.7 (GND), U3.0 (GND), X1.2, X1.4
- net VAA: now also C61.1, C62.1, C63.1, C64.1, C65.1, C66.1, C67.1, C68.1, C69.1, C70.1, C71.1
- net RXRF-: now reaches C34.1, L2.2, U1.5 (RXRF-)
- net RXRF+: now reaches C31.1, L2.1, U1.4 (RXRF+)
- net TXRF+: now reaches C36.1, L4.1, U1.10 (TXRF+)
- net TXRF-: now reaches C42.1, L4.2, U1.11 (TXRF-)
- net at PFIO1.15 (P15): now also R29.2
- net at PFIO1.17 (P17): now also R31.2
- net at PFIO1.19 (P19): now also R33.2
- net at PFIO1.21 (P21): now also R27.1
- net at R28.2: now also PFIO1.12 (P12); no longer PFIO1.22 (P22)
- net at PFIO1.24 (P24): no longer R29.2
- net at R30.2: now also PFIO1.14 (P14); no longer PFIO1.26 (P26)
- net at PFIO1.28 (P28): no longer R31.2
- net at R32.2: now also PFIO1.16 (P16); no longer PFIO1.30 (P30)
- net at PFIO1.32 (P32): no longer R33.2
- net at PFIO1.33 (P33): no longer R27.1
- net at R34.2: now also PFIO1.18 (P18); no longer PFIO1.34 (P34)
- new net 0V_dig: C11.2, C12.2, C13.2, C16.2, C17.2, C18.2, C19.2, C21.2, C22.2, C23.2, C24.2, C28.2, C29.2, C32.2, C44.2, C45.2, C46.2, C47.1, C48.1, C53.2, C54.2, C55.2, C56.2, C57.2, C58.2, C59.2, C60.2, C64.2, C66.2, C67.2, C7.2, D1.1 (A), D2.1 (A), P34.1 (P1), P38.2 (GND), P39.2 (GND), R23.2, R38.2, U2.0 (EP), U2.12 (GND), U2.17 (OGND), U2.37 (GND), U2.42 (GND), U2.5 (GND), U2.7 (GND), U3.0 (GND), X1.2, X1.4
- no-connect marks 45 -> 43
Other:
- note added: "vccrxlna \nbypass"
- moved on the sheet: C11, C12, C13, C14, C15, C16, C17, C18, C19, C20, C21, C22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

Commit message: bom, position files and gerbers generated
again
Parts:
- removed C70: 22pF, Capacitors_SMD:C_0402, symbol C
- removed C71: 10nF, Capacitors_SMD:C_0402, symbol C
- C72: renamed from 22pF1; value C_Small -> 22pF
- P10, P11, P12, P13, P14, P15, P16, P17, P18, P19, P20, P21, P22, P23, P24, P25, P26, P27, P28, P29, P3, P30, P31, P32, P33, P37, P4, P5, P6, P7, P8, P9: footprint hackrf1:GSG-TESTPOINT-30MIL-MASKONLY -> Connect:testpoint1mm
Connections:
- net 0V_dig: now also P29.1, P30.1, P31.1, P32.1
- net GND: no longer P29.1, P30.1, P31.1, P32.1
Other:
- moved on the sheet: C65, C68, C69

Commit message: version final antes de  planos de tierra
Parts:
- removed P10: TXENABLE, Connect:testpoint1mm, symbol CONN_1
- removed P16: DA0, Connect:testpoint1mm, symbol CONN_1
- removed P17: DA4, Connect:testpoint1mm, symbol CONN_1
- removed P18: DA7, Connect:testpoint1mm, symbol CONN_1
- removed P19: DD0, Connect:testpoint1mm, symbol CONN_1
- removed P20: DD5, Connect:testpoint1mm, symbol CONN_1
- removed P21: DD9, Connect:testpoint1mm, symbol CONN_1
- removed P29, P30, P31, P32: GND, Connect:testpoint1mm, symbol CONN_1
- removed P3: SCL, Connect:testpoint1mm, symbol CONN_1
- removed P37: INTR, Connect:testpoint1mm, symbol CONN_1
- removed P4: SDA, Connect:testpoint1mm, symbol CONN_1
- removed P5: SSP1_SCK, Connect:testpoint1mm, symbol CONN_1
- removed P6: SSP1_MOSI, Connect:testpoint1mm, symbol CONN_1
- removed P7: SSP1_MISO, Connect:testpoint1mm, symbol CONN_1
- removed P8: CS_XCVR, Connect:testpoint1mm, symbol CONN_1
- removed P9: CS_AD, Connect:testpoint1mm, symbol CONN_1
- C51: value 100pF -> 22pF; Description CAP CER 100PF 50V 5% NP0 0402 -> CAP CER 22PF 50V 5% NP0 0402; Note DNP -> (none); Part Number GRM1555C1H101JA01D -> GRM1555C1H220JA01D
- P2: footprint Pin_Headers:Pin_Header_Straight_1x02_Pitch3.96mm_Friction_Lock -> Pin_Headers:Pin_Header_Straight_2x01
Connections:
- net !VAA_ENABLE: now also PFIO2.23 (P23); no longer PSA1.25 (P25)
- net 0V_dig: now also C38.2, C39.2, C40.2, C41.2; no longer C58.2
- net CLK6: now also PFIO2.18 (P18); no longer PFIO2.16 (P16)
- net CS_XCVR: now also PSA1.6 (P6); no longer PSA1.12 (P12)
- net DA1: now also R33.1; no longer R34.1
- net DA2: now also R34.1; no longer R33.1
- net DA5: now also R30.2; no longer R30.1
- net DA7: now also R28.2; no longer R28.1
- net DD0: now also PFIO2.3 (P3); no longer PFIO1.13 (P13)
- net DD1: now also PFIO2.4 (P4); no longer PFIO1.10 (P10)
- net DD2: now also PFIO2.1 (P1); no longer PFIO1.8 (P8)
- net DD3: now also PFIO2.2 (P2); no longer PFIO1.7 (P7)
- net DD4: now also PFIO1.5 (P5); no longer PFIO1.6 (P6)
- net DD5: now also PFIO1.6 (P6); no longer PFIO1.5 (P5)
- net DD6: now also PFIO1.3 (P3); no longer PFIO1.4 (P4)
- net DD7: now also PFIO1.4 (P4); no longer PFIO1.3 (P3)
- net DD8: now also PFIO1.1 (P1); no longer PFIO1.2 (P2)
- net DD9: now also PFIO1.2 (P2); no longer PFIO1.1 (P1)
- net GND: now also C58.2, PSA1.23 (P23), PSA1.24 (P24); no longer C38.2, C39.2, C40.2, C41.2
- net GainCtrl_B1: now also PSA1.9 (P9); no longer PSA1.28 (P28)
- net GainCtrl_B2: now also PSA1.10 (P10); no longer PSA1.26 (P26)
- net GainCtrl_B3: now also PSA1.12 (P12); no longer PSA1.24 (P24)
- net GainCtrl_B4: now also PSA1.11 (P11); no longer PSA1.22 (P22)
- net GainCtrl_B5: now also PSA1.13 (P13); no longer PSA1.20 (P20)
- net GainCtrl_B7: now also PSA1.17 (P17); no longer PSA1.16 (P16)
- net INTR: now also PSA1.15 (P15)
- net MIX_CLK: now also P11.1; no longer PFIO2.18 (P18)
- net OEB: now also PSA1.28 (P28); no longer PSA1.21 (P21)
- net RXENABLE: now also PSA1.8 (P8); no longer P11.1, PSA1.9 (P9)
- net RXHP: now also PSA1.20 (P20); no longer PSA1.3 (P3)
- net SSP1_MISO: no longer C51.1
- net VAA: now also C51.1, D5.2 (A)
- net VCC: now also PSA1.27 (P27); no longer C25.1, C58.1, PFIO1.36 (P36), Q1.S, R1.1
- net XCVR_EN: now also PSA1.16 (P16); no longer D5.2 (A), PSA1.11 (P11)
- net at PFIO1.12 (P12): no longer R28.2
- net at PFIO1.14 (P14): no longer R30.2
- net at PFIO1.15 (P15): no longer R29.2
- net at PFIO1.16 (P16): no longer R32.2
- net at PFIO1.17 (P17): no longer R31.2
- net at PFIO1.18 (P18): no longer R34.2
- net at PFIO1.19 (P19): no longer R33.2
- net at PFIO1.21 (P21): no longer R27.1
- net at PFIO2.10 (P10): now also R31.2
- net at PFIO2.11 (P11): now also R32.2
- net at PFIO2.12 (P12): now also R34.2
- net at PFIO2.13 (P13): now also R33.2
- net at PFIO2.14 (P14): now also R27.1
- net at PFIO2.7 (P7): now also R28.1
- net at PFIO2.8 (P8): now also R29.2
- net at PFIO2.9 (P9): now also R30.1
- new net 3VDAC: C25.1, C58.1, PFIO1.36 (P36), Q1.S, R1.1
- no-connect marks 43 -> 42
Other:
- moved on the sheet: C58, P22, PFIO1, PFIO2, PSA1, R26, R27, R28, R29, R30, R31, R32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

Commit message: bypass capacitors y planos de tierra agregados
Parts:
- added C70, C71, C73, C74, C75: 2.2uF, Capacitors_SMD:C_0402, symbol C
Connections:
- net 0V_dig: now also C10.2, C14.2, C25.2, C30.2, C37.2, C51.2, C52.2, C58.2, C69.2, C8.2, C9.2, PSA1.23 (P23), PSA1.24 (P24), R14.1, R26.2, R37.2, R6.2, R7.2, R8.2, R9.2, C70.2, C71.2, C73.2, C74.2, C75.2
- net CLK5: now also P12.1
- net GND: no longer C10.2, C14.2, C20.2, C25.2, C30.2, C37.2, C51.2, C52.2, C58.2, C69.2, C8.2, C9.2, PSA1.23 (P23), PSA1.24 (P24), R14.1, R26.2, R37.2, R6.2, R7.2, R8.2, R9.2
- net VAA: no longer C20.1
- net VCC: now also C70.1, C71.1, C73.1, C74.1, C75.1
- net XTAL2: no longer P12.1
Other:
- moved on the sheet: C10, C14, C15, C2, C20, C22, C3, C4, C5, C57, C59, C6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

Commit message: text sixe and ground plane fixed,
Parts:
- P1, P34: footprint Connect:GSG-HOLE-06mm1 -> Connect:GSG-HOLE-06mm_nt
- PFIO1: footprint Socket_Strips:Socket_Strip_Straight_2x18 -> Socket_Strips:Socket_Strip_Straight_2x18_B
- PFIO2: footprint Socket_Strips:Socket_Strip_Straight_2x12 -> Socket_Strips:Socket_Strip_Straight_2x12_B
- PSA1: footprint Socket_Strips:Socket_Strip_Straight_2x14 -> Socket_Strips:Socket_Strip_Straight_2x14_B
Changed lines of the file:
@@
 F 0 "PSA1" H 10550 8650 50  0000 C CNN
 F 1 "CONN_02X14" V 10550 7900 50  0000 C CNN
-F 2 "Socket_Strips:Socket_Strip_Straight_2x14" H 10550 6750 60  0001 C CNN
+F 2 "Socket_Strips:Socket_Strip_Straight_2x14_B" H 10550 6750 60  0001 C CNN
 F 3 "" H 10550 6750 60  0000 C CNN
 	1    10550 7900
@@
 F 0 "PFIO1" H 15500 8650 50  0000 C CNN
 F 1 "CONN_02X18" V 15500 7700 50  0000 C CNN
-F 2 "Socket_Strips:Socket_Strip_Straight_2x18" H 15500 6650 60  0001 C CNN
+F 2 "Socket_Strips:Socket_Strip_Straight_2x18_B" H 15500 6650 60  0001 C CNN
 F 3 "" H 15500 6650 60  0000 C CNN
 	1    15500 7700
@@
 F 0 "P1" H 16300 1050 50  0000 C CNN
 F 1 "CONN_01X01" V 16400 950 50  0000 C CNN
-F 2 "Connect:GSG-HOLE-06mm1" H 16300 950 60  0001 C CNN
+F 2 "Connect:GSG-HOLE-06mm_nt" H 16300 950 60  0001 C CNN
 F 3 "" H 16300 950 60  0000 C CNN
 	1    16300 950
@@
 F 0 "P34" H 16200 2200 50  0000 C CNN
 F 1 "CONN_01X01" V 16300 2100 50  0000 C CNN
-F 2 "Connect:GSG-HOLE-06mm1" H 16200 2100 60  0001 C CNN
+F 2 "Connect:GSG-HOLE-06mm_nt" H 16200 2100 60  0001 C CNN
 F 3 "" H 16200 2100 60  0000 C CNN
 	1    16200 2100
@@
 F 0 "PFIO2" H 13300 8350 50  0000 C CNN
 F 1 "CONN_02X12" V 13300 7700 50  0000 C CNN
-F 2 "Socket_Strips:Socket_Strip_Straight_2x12" H 13300 6500 60  0001 C CNN
+F 2 "Socket_Strips:Socket_Strip_Straight_2x12_B" H 13300 6500 60  0001 C CNN
 F 3 "" H 13300 6500 60  0000 C CNN
 	1    13300 7700

Commit message: bom
Parts:
- C72: Description (none) -> CAP CER 22PF 50V 5% NP0 0402; Manufacturer (none) -> Murata; Part Number (none) -> GRM1555C1H220JA01D
- D3, D4, D5: Description (none) -> SMD CHIP LED 0603; Manufacturer (none) -> Kingbright; Part Number (none) -> APT1608SGC
- P1, P34: Note (none) -> DNP
- PFIO1: Description (none) -> 36P DR UNSHRD HRD .38 GOLD OVER NI; Manufacturer (none) -> Amphenol FCI; Part Number (none) -> 67996-236HLF
- PFIO2: Description (none) -> 24P DR UNSHRD HRD TIN OVER NI; Manufacturer (none) -> Amphenol FCI; Part Number (none) -> 67997-224HLF
- PSA1: Description (none) -> 28P DR UNSHRD HRD TIN OVER NI; Manufacturer (none) -> Amphenol FCI; Part Number (none) -> 67997-428HLF
- R27: Description (none) -> RES 0.0 OHM 1/16W 0402 SMD; Manufacturer (none) -> Stackpole; Part Number (none) -> RMCF0402ZT0R00
- R28, R29, R30, R31, R32, R33, R34: value R -> 0; Description (none) -> RES 0.0 OHM 1/16W 0402 SMD; Manufacturer (none) -> Stackpole; Part Number (none) -> RMCF0402ZT0R00
- T1: value RX_BALUN -> BALUN
- T2: value TX_BALUN -> BALUN
Connections:
- net 0V_dig is gone; now on net GND: C10.2, C11.2, C12.2, C13.2, C14.2, C16.2, C17.2, C18.2, C19.2, C21.2, C22.2, C23.2, C24.2, C25.2, C28.2, C29.2, C30.2, C32.2, C37.2, C38.2, C39.2, C40.2, C41.2, C44.2, C45.2, C46.2, C47.1, C48.1, C51.2, C52.2, C53.2, C54.2, C55.2, C56.2, C57.2, C58.2, C59.2, C60.2, C64.2, C66.2, C67.2, C69.2, C7.2, C70.2, C71.2, C73.2, C74.2, C75.2, C8.2, C9.2, D1.1 (A), D2.1 (A), P34.1 (P1), P38.2 (GND), P39.2 (GND), PSA1.23 (P23), PSA1.24 (P24), R14.1, R23.2, R26.2, R37.2, R38.2, R6.2, R7.2, R8.2, R9.2, U2.0 (EP), U2.12 (GND), U2.17 (OGND), U2.37 (GND), U2.42 (GND), U2.5 (GND), U2.7 (GND), U3.0 (GND), X1.2, X1.4
- net DA0: now also R27.1; no longer R27.2
- net DA1: now also R33.2; no longer R33.1
- net DA3: now also R32.2; no longer R32.1
- net GND: now also C20.2
- net VAA: now also C20.1
- net at PFIO2.11 (P11): now also R32.1; no longer R32.2
- net at PFIO2.13 (P13): now also R33.1; no longer R33.2
- net at PFIO2.14 (P14): now also R27.2; no longer R27.1
