File: HW/frontend/RFshield/Rfshield.kicad_pcb (KiCad board)
At the start: 4 copper layers, 73 x 50.9 mm, 306 parts, among them P10 TXENABLE, P11 RXENABLE, P13 GCK1, P16 DA0, P18 DA7, P2 VAA, P26 GND, P27 GND, P29 GND, P32 GND, P38 CLKIN, P39 CLKOUT, Q1 MOSFET_P, T1 RX_BALUN, T2 TX_BALUN, U1 MAX2837, U2 MAX5864, U3 SI5351C, X1 GSG-XTAL4PIN

Commit message: version final antes de  planos de tierra
Parts:
- removed 0Vdig, P32, gnd (x2): GND, Connect:testpoint1mm
- removed ? (x149): CONN_01X01, Connect:GSG-HOLE-06mm1
- removed ?: GND, Connect:1pin
- removed ?: CONN_01X01, Connect:GSG-HOLE-06mm
- removed C70: 10nF, Capacitors_SMD:C_0402
- removed C71: 22pF, Capacitors_SMD:C_0402
- removed P13: GCK1, Connect:testpoint1mm
- removed P16: DA0, Connect:testpoint1mm
- removed P18: DA7, Connect:testpoint1mm
- removed cs_ad: CS_AD, Connect:testpoint1mm
- removed gck2: GCK2, Connect:testpoint1mm
- removed gpioclk: SGPIO_CLK, Connect:testpoint1mm
- removed miso: SSP1_MISO, Connect:testpoint1mm
- removed mosi: SSP1_MOSI, Connect:testpoint1mm
- removed sck: SSP1_SCK, Connect:testpoint1mm
- removed scl: SCL, Connect:testpoint1mm
- removed sda: SDA, Connect:testpoint1mm
- added GndCon1: GND, Connect:1pin, F.Cu at (27.9, 112.6)
- C28, C29, C32, R17, R18, R19, R25: moved to B.Cu
- C51: value 100pF -> 22pF
- P2: footprint Pin_Headers:Pin_Header_Straight_1x02_Pitch3.96mm_Friction_Lock -> Pin_Headers:Pin_Header_Straight_2x01
- moved P29 51.0 mm to (23.1, 114.9)
- moved D5 49.6 mm to (72.3, 111.8), turned to 0 degrees
- moved R37 47.9 mm to (72.3, 113.7)
- moved D3 35.7 mm to (63.5, 72.4), turned to 270 degrees
- moved R35 33.6 mm to (63.5, 69.8), turned to 90 degrees
- moved C51 32.7 mm to (53.8, 85.9), turned to 0 degrees
- moved P11 22.9 mm to (46.5, 96.7)
- moved P27 15.9 mm to (52.6, 96.6)
- moved C38 14.6 mm to (71.3, 93.5)
- moved R25 14.2 mm to (30.5, 107.6), turned to 270 degrees
- moved C39 12.3 mm to (69.1, 93.5), turned to 180 degrees
- moved R36 11.5 mm to (31.8, 69.8), turned to 90 degrees
- moved R1 11.0 mm to (85.5, 113.3)
- moved C25 10.3 mm to (86.1, 111.4)
- moved C58 10.3 mm to (84.8, 111.4)
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Connections:
- C25 pad 1: VCC -> 3VDAC
- C38 pad 2: GND -> 0V_dig
- C39 pad 2: GND -> 0V_dig
- C40 pad 2: GND -> 0V_dig
- C41 pad 2: GND -> 0V_dig
- C51 pad 1: SSP1_MISO -> VAA
- C58 pad 1: VCC -> 3VDAC
- C58 pad 2: 0V_dig -> GND
- D5 pad 2: XCVR_EN -> VAA
- P11 pad 1: RXENABLE -> MIX_CLK
- PFIO1 pad 1: DD9 -> DD8
- PFIO1 pad 10: DD1 -> (no net)
- PFIO1 pad 12: Net-(PFIO1-Pad12) -> (no net)
- PFIO1 pad 13: DD0 -> (no net)
- PFIO1 pad 14: Net-(PFIO1-Pad14) -> (no net)
- PFIO1 pad 15: Net-(PFIO1-Pad15) -> (no net)
- PFIO1 pad 16: Net-(PFIO1-Pad16) -> (no net)
- PFIO1 pad 17: Net-(PFIO1-Pad17) -> (no net)
- PFIO1 pad 18: Net-(PFIO1-Pad18) -> (no net)
- PFIO1 pad 19: Net-(PFIO1-Pad19) -> (no net)
- PFIO1 pad 2: DD8 -> DD9
- PFIO1 pad 21: Net-(PFIO1-Pad21) -> (no net)
- PFIO1 pad 3: DD7 -> DD6
- PFIO1 pad 36: VCC -> 3VDAC
- PFIO1 pad 4: DD6 -> DD7
- PFIO1 pad 5: DD5 -> DD4
- PFIO1 pad 6: DD4 -> DD5
- PFIO1 pad 7: DD3 -> (no net)
- PFIO1 pad 8: DD2 -> (no net)
- PFIO2 pad 1: (no net) -> DD2
- PFIO2 pad 10: (no net) -> Net-(PFIO2-Pad10)
- PFIO2 pad 11: (no net) -> Net-(PFIO2-Pad11)
- PFIO2 pad 12: (no net) -> Net-(PFIO2-Pad12)
- PFIO2 pad 13: (no net) -> Net-(PFIO2-Pad13)
- PFIO2 pad 14: (no net) -> Net-(PFIO2-Pad14)
- PFIO2 pad 16: CLK6 -> (no net)
- PFIO2 pad 18: MIX_CLK -> CLK6
- PFIO2 pad 2: (no net) -> DD3
- PFIO2 pad 23: (no net) -> !VAA_ENABLE
- PFIO2 pad 3: (no net) -> DD0
- PFIO2 pad 4: (no net) -> DD1
- PFIO2 pad 7: (no net) -> Net-(PFIO2-Pad7)
- PFIO2 pad 8: (no net) -> Net-(PFIO2-Pad8)
- PFIO2 pad 9: (no net) -> Net-(PFIO2-Pad9)
- PSA1 pad 10: (no net) -> GainCtrl_B2
- PSA1 pad 11: XCVR_EN -> GainCtrl_B4
- PSA1 pad 12: CS_XCVR -> GainCtrl_B3
- PSA1 pad 13: (no net) -> GainCtrl_B5
- PSA1 pad 15: (no net) -> INTR
- PSA1 pad 16: GainCtrl_B7 -> XCVR_EN
- PSA1 pad 17: (no net) -> GainCtrl_B7
- PSA1 pad 20: GainCtrl_B5 -> RXHP
- PSA1 pad 21: OEB -> (no net)
- PSA1 pad 22: GainCtrl_B4 -> (no net)
- PSA1 pad 23: (no net) -> GND
- PSA1 pad 24: GainCtrl_B3 -> GND
- PSA1 pad 25: !VAA_ENABLE -> (no net)
- PSA1 pad 26: GainCtrl_B2 -> (no net)
- PSA1 pad 27: (no net) -> VCC
- PSA1 pad 28: GainCtrl_B1 -> OEB
- PSA1 pad 3: RXHP -> (no net)
- PSA1 pad 6: (no net) -> CS_XCVR
- PSA1 pad 8: (no net) -> RXENABLE
- PSA1 pad 9: RXENABLE -> GainCtrl_B1
- Q1 pad S: VCC -> 3VDAC
- R1 pad 1: VCC -> 3VDAC
- R19 pad 2: /INTR -> INTR
- R27 pad 1: Net-(PFIO1-Pad21) -> Net-(PFIO2-Pad14)
- R28 pad 1: DA7 -> Net-(PFIO2-Pad7)
- R28 pad 2: Net-(PFIO1-Pad12) -> DA7
- R29 pad 2: Net-(PFIO1-Pad15) -> Net-(PFIO2-Pad8)
- R30 pad 1: DA5 -> Net-(PFIO2-Pad9)
- R30 pad 2: Net-(PFIO1-Pad14) -> DA5
- R31 pad 2: Net-(PFIO1-Pad17) -> Net-(PFIO2-Pad10)
- R32 pad 2: Net-(PFIO1-Pad16) -> Net-(PFIO2-Pad11)
- R33 pad 1: DA2 -> DA1
- R33 pad 2: Net-(PFIO1-Pad19) -> Net-(PFIO2-Pad13)
- R34 pad 1: DA1 -> DA2
- R34 pad 2: Net-(PFIO1-Pad18) -> Net-(PFIO2-Pad12)
- U1 pad 16: /XCVR_CLKOUT -> (no net)
- U1 pad 32: RSSI -> (no net)
- U3 pad 3: /INTR -> INTR
Routing:
- net GND: track 137.0 -> 252.0 mm, vias 3 -> 27
- net 0V_dig: track 83.9 -> 172.5 mm, vias 1 -> 11
- net !VAA_ENABLE: track 73.6 -> 15.7 mm, vias 3 -> 1
- net VCC: track 131.5 -> 76.1 mm, vias 11 -> 5
- net SSP1_SCK: track 72.5 -> 110.1 mm, vias 3 -> 2
- net MIX_CLK: track 41.1 -> 7.29 mm
- net INTR: track 0.00 -> 33.5 mm, vias 0 -> 1
- net TXENABLE: track 75.1 -> 45.6 mm
- net SSP1_MOSI: track 101.6 -> 80.0 mm, vias 4 -> 2
- net RXENABLE: track 75.2 -> 54.5 mm
- net Net-(PFIO1-Pad17): track 19.0 -> 0.00 mm
- net GainCtrl_B1: track 43.1 -> 25.5 mm
- net Net-(PFIO1-Pad15): track 17.3 -> 0.00 mm, vias 1 -> 0
- net OEB: track 45.3 -> 28.1 mm, vias 3 -> 1
- net Net-(PFIO1-Pad19): track 17.1 -> 0.00 mm
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- removed copper zone on B.Cu, net 0V_dig
- removed copper zone on F.Cu, net 0V_dig
- removed copper zone on B.Cu, net GND
- removed copper zone on F.Cu, net GND
Other:
- net class Default: via_drill 0.4 -> 0.3
- net class vcc added: clearance 0.2, trace_width 0.4, via_dia 0.6, via_drill 0.4
