File: HW/frontend/RFshield/max2832version/RFshield/Rfshield.sch (KiCad schematic (older format))
At the start: 151 parts, among them P10 TXENABLE, P11 RXENABLE, P12 XTAL2, P13 GCK1, P14 GCK2, P15 SGPIO_CLK, P16 DA0, P17 DA4, P18 DA7, P19 DD0, P2 VAA, P20 DD5, P21 DD9, P22 RSSI, P23 GND, P24 GND, P25 GND, P26 GND, P27 GND, P28 GND, P29 GND, P3 SCL, P30 GND, P31 GND, P32 GND, P33 XCVR_CLKOUT, P37 INTR, P38 CLKIN, P39 CLKOUT, P4 SDA, P5 SSP1_SCK, P6 SSP1_MOSI, P7 SSP1_MISO, P8 CS_XCVR, P9 CS_AD, Q1 MOSFET_P, T1 RX_BALUN, T2 TX_BALUN, U1 MAX2832, U2 MAX5864, U3 SI5351C, X1 GSG-XTAL4PIN

Commit message: low budget version of rfshield netlisted
Connections:
- net !VAA_ENABLE: now also PSA1.25 (P25); no longer PSA1.1 (P1)
- net CS_AD: now also PSA1.5 (P5); no longer PSA1.2 (P2)
- net CS_XCVR: now also PSA1.12 (P12); no longer PSA1.4 (P4)
- net RXTXENABLE: now also PSA1.7 (P7); no longer PSA1.18 (P18)
- net SSP1_MISO: now also PSA1.1 (P1); no longer PSA1.11 (P11)
- net SSP1_MOSI: now also PSA1.4 (P4); no longer PSA1.12 (P12)
- net SSP1_SCK: now also PSA1.2 (P2); no longer PSA1.22 (P22)
- net XCVR_EN: now also PSA1.11 (P11); no longer PSA1.16 (P16)
- net ~shdn: now also PSA1.9 (P9); no longer PSA1.20 (P20)
Changed lines of the file:
@@
 Text GLabel 12550 7700 2    40   Input ~ 0
 SCL
+Text GLabel 12550 7600 2    40   Input ~ 0
+CS_XCVR
 Text GLabel 12550 7200 2    40   Input ~ 0
-CS_XCVR
-Text GLabel 12550 7600 2    40   Input ~ 0
 SSP1_MOSI
-Text GLabel 11850 7600 0    40   Input ~ 0
+Text GLabel 11850 7100 0    40   Input ~ 0
 SSP1_MISO
-Text GLabel 12550 8100 2    40   Input ~ 0
+Text GLabel 12550 7100 2    40   Input ~ 0
 SSP1_SCK
 $Comp
@@
 	1    0    0    -1
 $EndComp
-Text GLabel 12550 7800 2    40   Input ~ 0
+Text GLabel 11850 7600 0    40   Input ~ 0
 XCVR_EN
-Text GLabel 12550 8000 2    40   Input ~ 0
+Text GLabel 11850 7500 0    40   Input ~ 0
 ~shdn
-Text GLabel 12550 7900 2    40   Input ~ 0
+Text GLabel 11850 7400 0    40   Input ~ 0
 RXTXENABLE
-Text GLabel 12550 7100 2    40   Input ~ 0
+Text GLabel 11850 7300 0    40   Input ~ 0
 CS_AD
 Text Notes 12400 7000 0    60   ~ 0
@@
 Wire Wire Line
 	11800 8000 11950 8000
-Wire Wire Line
-	11850 7600 11950 7600
-Wire Wire Line
-	12550 7100 12450 7100
-Wire Wire Line
-	12550 7200 12450 7200
-Wire Wire Line
-	12550 7600 12450 7600
-Wire Wire Line
-	12550 8100 12450 8100
 Wire Notes Line
 	12950 7050 12950 7250
@@
 Wire Notes Line
 	12500 7750 13000 7750
-Wire Wire Line
-	12550 7800 12450 7800
-Wire Wire Line
-	12550 7900 12450 7900
-Wire Wire Line
-	12550 8000 12450 8000
 $Comp
 L GND #PWR104
@@
 Wire Wire Line
 	14100 8700 14250 8700
-NoConn ~ 11950 7200
-NoConn ~ 11950 7300
-NoConn ~ 11950 7400
-NoConn ~ 11950 7500
 NoConn ~ 12450 7300
 NoConn ~ 12450 7400
@@
 NoConn ~ 11950 7900
 NoConn ~ 11950 8200
-NoConn ~ 11950 8300
 NoConn ~ 11950 8400
 NoConn ~ 12450 8200
@@
 Wire Wire Line
 	15800 1300 15800 1400
-Text GLabel 11850 7100 0    40   Input ~ 0
+Text GLabel 11850 8300 0    40   Input ~ 0
 !VAA_ENABLE
-Wire Wire Line
-	11850 7100 11950 7100
 Wire Wire Line
 	11700 950  11700 900
@@
 Wire Wire Line
 	7250 3550 7250 3650
+Wire Wire Line
+	11850 8300 11950 8300
+Wire Wire Line
+	11850 7100 11950 7100
+Wire Wire Line
+	11850 7300 11950 7300
+NoConn ~ 11950 7200
+Wire Wire Line
+	11850 7400 11950 7400
+Wire Wire Line
+	11850 7600 11950 7600
+Wire Wire Line
+	11850 7500 11950 7500
+Wire Wire Line
+	12450 7200 12550 7200
+Wire Wire Line
+	12550 7600 12450 7600
+Wire Wire Line
+	12450 7100 12550 7100
+NoConn ~ 12450 8100
+NoConn ~ 12450 8000
+NoConn ~ 12450 7900
+NoConn ~ 12450 7800
 $EndSCHEMATC
